File: mpcie-breakout.brd (EAGLE design)
At the start: 70 x 70 mm, 43 parts, among them K1 694108106102, U1 IP4234CZ6, U2 LD1085D2T33R, X1 MPCIE-JAE, X2 MINI-USB-SHIELD-UX60-MB-5ST

Commit message: added RXD, TXD, RTS, CTS
Connections:
- net REFCLK+ renamed RTS_3.3V
- net REFCLK- renamed CTS_3.3V
- net UIM_C4 renamed TXD_3.3V
- net UIM_C8 renamed RXD_3.3V
Changed lines of the file:
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@@
 <wire x1="38.42" y1="54.544" x2="38.42" y2="54.247" width="0.5" layer="16"/>
 </signal>
-<signal name="UIM_C8">
+<signal name="RXD_3.3V">
 <contactref element="X1" pad="17"/>
 <contactref element="JP4" pad="7"/>
@@
 <wire x1="14.111875" y1="58.786125" x2="14.111875" y2="58.71" width="0.3048" layer="16"/>
 </signal>
-<signal name="UIM_C4">
+<signal name="TXD_3.3V">
 <contactref element="X1" pad="19"/>
 <contactref element="JP4" pad="10"/>
@@
 <wire x1="6.911875" y1="62.176125" x2="6.911875" y2="58.71" width="0.3048" layer="16"/>
 </signal>
-<signal name="REFCLK-">
+<signal name="CTS_3.3V">
 <contactref element="X1" pad="11"/>
 <contactref element="JP4" pad="5"/>
@@
 <wire x1="8.511875" y1="62.100125" x2="8.511875" y2="58.71" width="0.3048" layer="16"/>
 </signal>
-<signal name="REFCLK+">
+<signal name="RTS_3.3V">
 <contactref element="X1" pad="13"/>
 <contactref element="JP4" pad="8"/>
